Commit message: gazebo sim changes

File: src/my_bot/description/camera.xacro (robot description, xacro)
@@ -11,5 +11,12 @@
                 <box size="0.010 0.03 0.03"/>
             </geometry>
-            <material name="lime"/>
+            <material name="black"/>
+        </visual>
+        <visual>
+            <origin xyz="0 0 -0.05"/>
+            <geometry>
+                <cylinder radius="0.002" length="0.1"/>
+            </geometry>
+            <material name="green"/>
         </visual>
     </link>
@@ -21,5 +28,5 @@
     <link name="camera_link_optical"></link>
     <gazebo reference="camera_link">
-        <material>Gazebo/Green</material>
+        <material>Gazebo/black</material>
         <sensor name = "camera" type = "camera">
             <always_on>true</always_on>
@@ -27,6 +34,6 @@
             <visualize>true</visualize>
             <update_rate>10</update_rate>
-            <topic>camera/image_raw</topic> <gz_frame_id>camera_link_optical</gz_frame_id>
             <camera>
+                <camera_info_topic>camera/camera_info</camera_info_topic>
                 <horizontal_fov>1.089</horizontal_fov>
                 <image>
@@ -40,4 +47,9 @@
                 </clip>
             </camera>
+            <plugin name="camera_controller" filename="libgazebo_ros_camera.so">
+                <frame_name>camera_link_optical</frame_name>
+            </plugin>
+            <topic>camera/image_raw</topic>
+            <get_frame_id>camera_link_optical</get_frame_id>
         </sensor>
     </gazebo>

File: src/my_bot/description/colors.xacro (robot description, xacro)
@@ -7,6 +7,6 @@
         <color rgba="0.3 0.3 0.3 1"/>
     </material>
-    <material name="lime">
-        <color rgba="0.6 1 0.2 1"/>
+    <material name="green">
+        <color rgba="0 1 0 1"/>
     </material>
     <material name="gold">
@@ -16,3 +16,6 @@
         <color rgba="1 0 0 1"/>
     </material>
+    <material name="black">
+        <color rgba="0 0 0 1"/>
+    </material>
 </robot>

File: src/my_bot/description/gazebo_control.xacro (robot description, xacro)
@@ -6,10 +6,18 @@
             <right_joint>right_wheel_joint</right_joint>
             <wheel_separation>0.35</wheel_separation>
-            <wheel_radius>0.05</wheel_radius> <topic>cmd_vel</topic>
-            <odom_topic>model/my_bot/odometry</odom_topic>
-            <tf_topic>model/my_bot/tf</tf_topic>
+            <wheel_radius>0.033</wheel_radius>
+            <max_linear_acceleration>0.33</max_linear_acceleration>
+            <topic>cmd_vel</topic>
             <frame_id>odom</frame_id>
             <child_frame_id>base_link</child_frame_id>
-            <max_linear_acceleration>10.0</max_linear_acceleration>
+            <odom_topic>odom</odom_topic>
+            <odom_publisher_frequency>30</odom_publisher_frequency>
+            <tf_topic>/tf</tf_topic>
+        </plugin>
+        <plugin filename="gz-sim-joint-state-publisher-system"
+            name="gz::sim::systems::JointStatePublisher">
+            <topic>joint_states</topic>
+            <joint_name>left_wheel_joint</joint_name>
+            <joint_name>right_wheel_joint</joint_name>
         </plugin>
     </gazebo>

File: src/my_bot/description/lidar.xacro (robot description, xacro)
@@ -42,5 +42,5 @@
                 </range>
             </lidar>
-            <topic>model/my_bot/scan</topic>
+            <topic>scan</topic>
             <gz_frame_id>laser_frame</gz_frame_id>
         </sensor>

Commit message: updated bridge.yaml, removed joint pub

File: src/my_bot/description/camera.xacro (robot description, xacro)
@@ -14,7 +14,7 @@
         </visual>
         <visual>
-            <origin xyz="0 0 -0.05"/>
+            <origin xyz="0.005 0 0" rpy="0 ${pi/2} 0"/>
             <geometry>
-                <cylinder radius="0.002" length="0.1"/>
+                <cylinder radius="0.005" length="0.005"/>
             </geometry>
             <material name="green"/>

Commit message: slam teleop working

File: src/my_bot/description/camera.xacro (robot description, xacro)
@@ -47,7 +47,4 @@
                 </clip>
             </camera>
-            <plugin name="camera_controller" filename="libgazebo_ros_camera.so">
-                <frame_name>camera_link_optical</frame_name>
-            </plugin>
             <topic>camera/image_raw</topic>
             <get_frame_id>camera_link_optical</get_frame_id>

File: src/my_bot/description/gazebo_control.xacro (robot description, xacro)
@@ -2,5 +2,5 @@
 <robot xmlns:xacro="http://www.ros.org/wiki/xacro">
     <gazebo>
-        <plugin filename="gz-sim-diff-drive-system" name="gz::sim::systems::DiffDrive">
+        <plugin name="gz::sim::systems::DiffDrive" filename="gz-sim-diff-drive-system">
             <left_joint>left_wheel_joint</left_joint>
             <right_joint>right_wheel_joint</right_joint>

File: src/my_bot/description/lidar.xacro (robot description, xacro)
@@ -38,6 +38,6 @@
                 </scan>
                 <range>
-                    <min>0.3</min>
-                    <max>12</max>
+                    <min>0.0</min>
+                    <max>25</max>
                 </range>
             </lidar>

File: src/my_bot/description/robot.urdf.xacro (robot description, xacro)
@@ -1,8 +1,17 @@
 <?xml version="1.0"?>
 <robot xmlns:xacro="http://www.ros.org/wiki/xacro"  name="robot">
+    <xacro:arg name = "use_ros2_control" default = "true"/>
     <!-- Example link -->
     <xacro:include filename="robot_core.xacro"/>
-    <xacro:include filename="gazebo_control.xacro"/>
+    <!-- <xacro:include filename="gazebo_control.xacro"/> -->
     <xacro:include filename="lidar.xacro"/>
     <xacro:include filename="camera.xacro"/>
+    <!-- <xacro:include filename="ros2_control.xacro"/> -->
+    <!-- Switch between ros2_control and Gazebo integrated diff-drive control -->
+    <xacro:if value="$(arg use_ros2_control)">
+        <xacro:include filename="ros2_control.xacro" />
+    </xacro:if>
+    <xacro:unless value="$(arg use_ros2_control)">
+        <xacro:include filename="gazebo_control.xacro" />
+    </xacro:unless>
 </robot>

File: src/my_bot/description/robot_core.xacro (robot description, xacro)
@@ -21,4 +21,12 @@
         <origin xyz="-0.1 0 0"/>
     </joint>
+        <!-- BASE_FOOTPRINT -->
+    <joint name="base_footprint_joint" type="fixed">
+        <parent link="base_link"/>
+        <child link="base_footprint"/>
+        <origin xyz="0 0 0" rpy="0 0 0"/>
+    </joint>
+    <link name="base_footprint">
+    </link>
     <link name="chassis">
         <visual>
