Commit message: control by teleop

File: src/my_bot/description/lidar.xacro (robot description, xacro)
@@ -24,5 +24,5 @@
     <gazebo reference="laser_frame">
         <material>Gazebo/Red</material>
-        <sensor name="laser" type="ray">
+        <sensor name="laser" type="gpu_ray">
             <pose> 0 0 0 0 0 0 </pose>
             <visualize>true</visualize>
@@ -41,12 +41,5 @@
                 </range>
             </ray>
-            <plugin name="laser_controller" filename="libgazebo_ros_ray_sensor.so">
-                <ros>
-                    <argument>~/out:=scan</argument>
-                </ros>
-                <output_type>sensor_msgs/LaserScan</output_type>
-                <frame_name>laser_frame</frame_name>
-            </plugin>
-        </sensor>
+            </sensor>
     </gazebo>
 </robot>

File: src/my_bot/description/robot_core.xacro (robot description, xacro)
@@ -2,23 +2,18 @@
 <robot xmlns:xacro="http://www.ros.org/wiki/xacro"  name="robot">
     <xacro:include filename="inertial_macros.xacro"/>
-    <material name="cyan">
-        <color rgba="0 1 1 1"/>
-    </material>
-    <material name="metal_gray">
-        <color rgba="0.3 0.3 0.3 1"/>
-    </material>
-    <material name="lime">
-        <color rgba="0.6 1 0.2 1"/>
-    </material>
-    <material name="gold">
-        <color rgba="1 0.84 0 1"/>
-    </material>
-    <material name="red">
-        <color rgba="1 0 0 1"/>
-    </material>
-    <!-- BASE LINK -->
+    <xacro:include filename="colors.xacro"/>
+    <xacro:property name="chassis_length" value="0.3"/>
+    <xacro:property name="chassis_width" value="0.3"/>
+    <xacro:property name="chassis_height" value="0.15"/>
+    <xacro:property name="chassis_mass" value="0.5"/>
+    <xacro:property name="wheel_radius" value="0.05"/>
+    <xacro:property name="wheel_thickness" value="0.04"/>
+    <xacro:property name="wheel_mass" value="0.1"/>
+    <xacro:property name="wheel_offset_y" value="0.175"/>
+    <xacro:property name="caster_wheel_radius" value="0.05"/>
+    <xacro:property name="caster_wheel_mass" value="0.1"/>
+    <xacro:property name="caster_wheel_offset_x" value="0.24"/>
     <link name="base_link">
     </link>
-    <!-- CHASSIS -->
     <joint name="chassis_joint" type="fixed">
         <parent link="base_link"/>
@@ -28,25 +23,24 @@
     <link name="chassis">
         <visual>
-            <origin xyz="0.15 0 0.075" rpy="0 0 0"/>
+            <origin xyz="${chassis_length/2} 0 ${chassis_height/2}" rpy="0 0 0"/>
             <geometry>
-                <box size="0.3 0.3 0.15"/>
+                <box size="${chassis_length} ${chassis_width} ${chassis_height}"/>
             </geometry>
             <material name="metal_gray"/>
         </visual>
         <collision>
-            <origin xyz="0.15 0 0.075" rpy="0 0 0"/>
+            <origin xyz="${chassis_length/2} 0 ${chassis_height/2}" rpy="0 0 0"/>
             <geometry>
-                <box size="0.3 0.3 0.15"/>
+                <box size="${chassis_length} ${chassis_width} ${chassis_height}"/>
             </geometry>
         </collision>
-        <xacro:inertial_box mass="0.5" x="0.3" y="0.3" z="0.15">
-            <origin xyz="0.15 0 0.075" rpy="0 0 0"/>
+        <xacro:inertial_box mass="${chassis_mass}" x="${chassis_length}" y="${chassis_width}" z="${chassis_height}">
+            <origin xyz="${chassis_length/2} 0 ${chassis_height/2}" rpy="0 0 0"/>
         </xacro:inertial_box>
     </link>
-    <!-- LEFT WHEEL -->
     <joint name="left_wheel_joint" type="continuous">
         <parent link="base_link"/>
         <child link="left_wheel"/>
-        <origin xyz="0 0.175 0" rpy="-${pi/2} 0 0"/>
+        <origin xyz="0 ${wheel_offset_y} 0" rpy="-${pi/2} 0 0"/>
         <axis xyz="0 0 1"/>
     </joint>
@@ -54,5 +48,5 @@
         <visual>
             <geometry>
-                <cylinder length="0.04" radius="0.05" />
+                <cylinder length="${wheel_thickness}" radius="${wheel_radius}" />
             </geometry>
             <material name="gold"/>
@@ -60,16 +54,15 @@
         <collision>
             <geometry>
-                <cylinder length="0.04" radius="0.05" />
+                <cylinder length="${wheel_thickness}" radius="${wheel_radius}" />
             </geometry>
         </collision>
-        <xacro:inertial_cylinder mass="0.1" length="0.05" radius="0.05">
+        <xacro:inertial_cylinder mass="${wheel_mass}" length="${wheel_thickness}" radius="${wheel_radius}">
             <origin xyz="0 0 0" rpy="0 0 0"/>
         </xacro:inertial_cylinder>
     </link>
-    <!-- RIGHT WHEEL -->
     <joint name="right_wheel_joint" type="continuous">
         <parent link="base_link"/>
         <child link="right_wheel"/>
-        <origin xyz="0 -0.175 0" rpy="${pi/2} 0 0"/>
+        <origin xyz="0 -${wheel_offset_y} 0" rpy="${pi/2} 0 0"/>
         <axis xyz="0 0 -1"/>
     </joint>
@@ -77,5 +70,5 @@
         <visual>
             <geometry>
-         <cylinder length="0.04" radius="0.05" />
+                <cylinder length="${wheel_thickness}" radius="${wheel_radius}" />
             </geometry>
             <material name="gold"/>
@@ -83,21 +76,20 @@
         <collision>
             <geometry>
-                <cylinder length="0.04" radius="0.05" />
+                <cylinder length="${wheel_thickness}" radius="${wheel_radius}" />
             </geometry>
         </collision>
-        <xacro:inertial_cylinder mass="0.1" length="0.05" radius="0.05">
+        <xacro:inertial_cylinder mass="${wheel_mass}" length="${wheel_thickness}" radius="${wheel_radius}">
             <origin xyz="0 0 0" rpy="0 0 0"/>
         </xacro:inertial_cylinder>
     </link>
-    <!-- CASTER WHEEL -->
     <joint name="caster_wheel_joint" type="fixed">
         <parent link="chassis"/>
         <child link="caster_wheel"/>
-        <origin xyz="0.24 0 0" rpy="0 0 0"/>
+        <origin xyz="${caster_wheel_offset_x} 0 0" rpy="0 0 0"/>
     </joint>
     <link name="caster_wheel">
         <visual>
             <geometry>
-                <sphere radius="0.05" />
+                <sphere radius="${caster_wheel_radius}" />
             </geometry>
             <material name="cyan"/>
@@ -105,12 +97,12 @@
         <collision>
             <geometry>
-                <sphere radius="0.05" />
+                <sphere radius="${caster_wheel_radius}" />
             </geometry>
         </collision>
-        <xacro:inertial_sphere mass="0.1" radius="0.05">
+        <xacro:inertial_sphere mass="${caster_wheel_mass}" radius="${caster_wheel_radius}">
             <origin xyz="0 0 0" rpy="0 0 0"/>
         </xacro:inertial_sphere>
     </link>
-    <gazebo reference = "caster_wheel">
+    <gazebo reference="caster_wheel">
         <mu1 value="0.001"/>
         <mu2 value="0.001"/>

Commit message: nav2 working

File: src/my_bot/description/lidar.xacro (robot description, xacro)
@@ -28,5 +28,5 @@
             <pose> 0 0 0 0 0 0 </pose>
             <visualize>true</visualize>
-            <update_rate>10</update_rate>
+            <update_rate>30</update_rate>
             <lidar>
                 <scan>

File: src/my_bot/description/robot_core.xacro (robot description, xacro)
@@ -6,19 +6,16 @@
     <xacro:property name="chassis_width" value="0.3"/>
     <xacro:property name="chassis_height" value="0.15"/>
-    <xacro:property name="chassis_mass" value="0.5"/>
+    <!-- <xacro:property name="chassis_mass" value="0.5"/> -->
+     <xacro:property name="chassis_mass" value="1.0"/>
     <xacro:property name="wheel_radius" value="0.05"/>
     <xacro:property name="wheel_thickness" value="0.04"/>
-    <xacro:property name="wheel_mass" value="0.1"/>
+    <xacro:property name="wheel_mass" value="0.05"/>
+     <!-- <xacro:property name="wheel_mass" value="0.1"/> -->
     <xacro:property name="wheel_offset_y" value="0.175"/>
     <xacro:property name="caster_wheel_radius" value="0.05"/>
-    <xacro:property name="caster_wheel_mass" value="0.1"/>
+    <xacro:property name="caster_wheel_mass" value="0.5"/>
     <xacro:property name="caster_wheel_offset_x" value="0.24"/>
     <link name="base_link">
     </link>
-    <joint name="chassis_joint" type="fixed">
-        <parent link="base_link"/>
-        <child link="chassis"/>
-        <origin xyz="-0.1 0 0"/>
-    </joint>
         <!-- BASE_FOOTPRINT -->
     <joint name="base_footprint_joint" type="fixed">
@@ -29,4 +26,9 @@
     <link name="base_footprint">
     </link>
+    <joint name="chassis_joint" type="fixed">
+        <parent link="base_link"/>
+        <child link="chassis"/>
+        <origin xyz="-0.1 0 0"/>
+    </joint>
     <link name="chassis">
         <visual>
